File: PCB/EMP_Cyclone_SAO_v1/EMP_Cyclone_SAO_v1.kicad_sch (KiCad schematic)
At the start: 6 parts, among them SW1 SW_Push, SW2 SW_Push, SW3 SW_Push

Commit message: updated to use ESP32-C3 supermini
Parts:
- removed A1: Arduino_Nano_Every, PCM_arduino-library:Arduino_Nano_Every_Tile, symbol MCU_Module:Arduino_Nano_Every
- added U3: ESP32-C3_SUPERMINI, neopixelrings-2:MODULE_ESP32-C3_SUPERMINI, symbol neopixel_ring_16:ESP32-C3_SUPERMINI
Connections:
- net +5V: now also U1. (GND), U2. (GND), U3.5V
- net GND: now also U3.G (GND)
- net at SW2.1: now also U3.4 (GPIO4)
- net at SW3.1: now also U3.6 (GPIO6)
- net at SW1.1: now also U3.5 (GPIO5)
- new net: U1. (GND), U2. (GND)
- new net: U2. (GND), U3.2 (GPIO2)

Commit message: Update files in prep for moving repo
Parts:
- removed SW3: SW_Push, Button_Switch_THT:SW_PUSH_6mm, symbol Switch:SW_Push
Connections:
- new net: U1. (GND), U2. (GND)
Changed lines of the file:
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@@
 	(paper "A4")
-	(junction
-		(at 81.28 157.48)
-		(diameter 0)
-		(color 0 0 0 0)
-	)
 	(junction
 		(at 81.28 134.62)
@@
 	(wire
 		(pts
-			(xy 69.85 157.48) (xy 81.28 157.48)
-		)
-		(stroke
-			(width 0)
-			(type default)
-		)
-	)
-	(wire
-		(pts
 			(xy 81.28 160.02) (xy 167.64 160.02)
 		)
@@
 	(wire
 		(pts
-			(xy 59.69 157.48) (xy 57.15 157.48)
-		)
-		(stroke
-			(width 0)
-			(type default)
-		)
-	)
-	(wire
-		(pts
 			(xy 142.24 44.45) (xy 142.24 109.22)
 		)
@@
 	(wire
 		(pts
-			(xy 57.15 101.6) (xy 68.58 101.6)
-		)
-		(stroke
-			(width 0)
-			(type default)
-		)
-	)
-	(wire
-		(pts
 			(xy 69.85 134.62) (xy 81.28 134.62)
 		)
@@
 	(wire
 		(pts
-			(xy 81.28 146.05) (xy 81.28 157.48)
-		)
-		(stroke
-			(width 0)
-			(type default)
-		)
-	)
-	(wire
-		(pts
 			(xy 106.68 81.28) (xy 138.43 81.28)
 		)
@@
 	(wire
 		(pts
-			(xy 81.28 157.48) (xy 81.28 160.02)
+			(xy 81.28 146.05) (xy 81.28 160.02)
 		)
 		(stroke
@@
 		(pts
 			(xy 106.68 151.13) (xy 134.62 151.13)
-		)
-		(stroke
-			(width 0)
-			(type default)
-		)
-	)
-	(wire
-		(pts
-			(xy 57.15 157.48) (xy 57.15 101.6)
 		)
 		(stroke
@@
 					(unit 1)
 				)
-			)
-		)
-	)
-	(symbol
-		(lib_id "Switch:SW_Push")
-		(at 64.77 157.48 0)
-		(unit 1)
-		(exclude_from_sim no)
-		(in_bom yes)
-		(on_board yes)
-		(dnp no)
-		(property "Reference" "SW3"
-			(at 64.77 149.86 0)
-			(effects
-				(font
-					(size 1.27 1.27)
-				)
-			)
-		)
-		(property "Value" "SW_Push"
-			(at 64.77 152.4 0)
-			(effects
-				(font
-					(size 1.27 1.27)
-				)
-			)
-		)
-		(property "Footprint" "Button_Switch_THT:SW_PUSH_6mm"
-			(at 64.77 152.4 0)
-			(effects
-				(font
-					(size 1.27 1.27)
-				)
-				(hide yes)
-			)
-		)
-		(property "Datasheet" "~"
-			(at 64.77 152.4 0)
-			(effects
-				(font
-					(size 1.27 1.27)
-				)
-				(hide yes)
-			)
-		)
-		(property "Description" "Push button switch, generic, two pins"
-			(at 64.77 157.48 0)
-			(effects
-				(font
-					(size 1.27 1.27)
-				)
-				(hide yes)
-			)
-		)
-		(pin "1"
-		)
-		(pin "2"
-		)
-		(instances
-			(project "EMP_Cyclone_SAO_v1"
-				(path "/5abfebdb-db98-4538-9b9b-a79c9de2c6a9"
-					(reference "SW3")
-					(unit 1)
-				)
